Commit message: training,deploy: align physics with calibrated vehicle
Co-authored-by: Cursor <cursoragent@cursor.com>

File: training/F110.export.urdf (robot description, URDF)
Before this commit: robot racecar, 13 links, 12 joints
Links:
- link left_front_wheel: geometry collision cylinder length=0.045 radius=0.053; visual mesh filename=f1tenth_model/meshes/left_front_wheel.STL
- link left_rear_wheel: geometry collision cylinder length=0.045 radius=0.053; visual mesh filename=f1tenth_model/meshes/left_rear_wheel.STL
- link right_front_wheel: geometry collision cylinder length=0.045 radius=0.053; visual mesh filename=f1tenth_model/meshes/right_front_wheel.STL
- link right_rear_wheel: geometry collision cylinder length=0.045 radius=0.053; visual mesh filename=f1tenth_model/meshes/right_rear_wheel.STL
Joints:
- joint left_rear_wheel_joint: origin xyz=0 0.1 0 rpy=1.5708 0 0 -> xyz=0 0.1265 0 rpy=1.5708 0 0
- joint left_steering_hinge_joint: origin xyz=0.325 0.1 0 rpy=0 1.5708 0 -> xyz=0.325 0.1265 0 rpy=0 1.5708 0
- joint right_rear_wheel_joint: origin xyz=0 -0.1 0 rpy=1.5708 0 0 -> xyz=0 -0.1265 0 rpy=1.5708 0 0
- joint right_steering_hinge_joint: origin xyz=0.325 -0.1 0 rpy=0 1.5708 0 -> xyz=0.325 -0.1265 0 rpy=0 1.5708 0
